Commit message: revitalise pitek->twins 2

File: urdf/lbr4/lbr.urdf.xacro (robot description, xacro)
@@ -1,6 +1,4 @@
 <?xml version="1.0"?>
 <robot xmlns:xacro="http://www.ros.org/wiki/xacro">
-  <xacro:include filename="$(find pitasc_robot_descriptions)/urdf/lbr4/lbr.gazebo.xacro" />
-  <xacro:include filename="$(find pitasc_robot_descriptions)/urdf/lbr4/lbr.transmission.xacro" />
   <xacro:property name="pi" value="3.14159265" />
   <xacro:macro name="lbr4" params="prefix parent r:=1.0 g:=0.5 b:=0.0 *origin">
@@ -21,5 +19,5 @@
           <cylinder radius="0.060" length="0.12"/>
         </geometry>
-        <material name="lbr-material">
+        <material name="${prefix}-material">
           <color rgba="${r} ${g} ${b} 1.0"/>
         </material>
@@ -54,5 +52,5 @@
           <mesh filename="package://pitasc_robot_descriptions/meshes/lbr4/joint_1.stl" />
         </geometry>
-        <material name="lbr-material" />
+        <material name="${prefix}-material" />
       </visual>
       <collision>
@@ -84,5 +82,5 @@
           <mesh filename="package://pitasc_robot_descriptions/meshes/lbr4/joint_2.stl" />
         </geometry>
-        <material name="lbr-material" />
+        <material name="${prefix}-material" />
       </visual>
       <collision>
@@ -114,5 +112,5 @@
           <mesh filename="package://pitasc_robot_descriptions/meshes/lbr4/joint_3.stl" />
         </geometry>
-        <material name="lbr-material" />
+        <material name="${prefix}-material" />
       </visual>
       <collision>
@@ -145,5 +143,5 @@
           <mesh filename="package://pitasc_robot_descriptions/meshes/lbr4/joint_4.stl" />
         </geometry>
-        <material name="lbr-material" />
+        <material name="${prefix}-material" />
       </visual>
       <collision>
@@ -174,5 +172,5 @@
           <mesh filename="package://pitasc_robot_descriptions/meshes/lbr4/joint_5.stl" />
         </geometry>
-        <material name="lbr-material" />
+        <material name="${prefix}-material" />
       </visual>
       <collision>
@@ -204,5 +202,5 @@
           <mesh filename="package://pitasc_robot_descriptions/meshes/lbr4/joint_6.stl" />
         </geometry>
-        <material name="lbr-material" />
+        <material name="${prefix}-material" />
       </visual>
       <collision>
@@ -234,5 +232,5 @@
           <mesh filename="package://pitasc_robot_descriptions/meshes/lbr4/joint_7.stl" />
         </geometry>
-        <material name="lbr-material" />
+        <material name="${prefix}-material" />
       </visual>
       <collision>
@@ -250,7 +248,4 @@
     </joint>
     <link name="${prefix}ee"/>
-    <!-- extensions -->
-    <xacro:lbr_gazebo name="${prefix}" />
-    <xacro:lbr_transmission name="${prefix}" />
   </xacro:macro>
 </robot>
