Commit message: add simple box xacro (typical adapter plate)

File: urdf/utils/box.urdf.xacro (robot description, xacro)
@@ -59,3 +59,28 @@
     <link name="${prefix}center_top"/>
   </xacro:macro>
+  <xacro:macro name="simple_box" params="prefix parent *origin
+    length width height *color">
+    <joint name="${prefix}floor_joint" type="fixed">
+      <parent link="${parent}"/>
+      <child link="${prefix}floor"/>
+      <xacro:insert_block name="origin" />
+    </joint>
+    <link name="${prefix}floor">
+        <visual>
+            <geometry>
+                <box size="${length} ${width} ${height}"/>
+            </geometry>
+            <origin rpy="0 0 0" xyz="0 0 ${height/2}"/>
+            <material name="${prefix}color">
+              <xacro:insert_block name="color" />
+            </material>
+        </visual>
+    </link>
+    <joint name="${prefix}center_top_jnt" type="fixed">
+      <origin xyz="0 0 ${height}" rpy="0 0 0"/>
+      <parent link="${prefix}floor"/>
+      <child link="${prefix}center_top"/>
+    </joint>
+    <link name="${prefix}center_top"/>
+  </xacro:macro>
 </robot>

Commit message: add minimal box with only one link

File: urdf/utils/box.urdf.xacro (robot description, xacro)
@@ -84,3 +84,22 @@
     <link name="${prefix}center_top"/>
   </xacro:macro>
+  <xacro:macro name="minimal_box" params="prefix parent *origin
+    length width height *color">
+    <joint name="${prefix}floor_joint" type="fixed">
+      <parent link="${parent}"/>
+      <child link="${prefix}floor"/>
+      <xacro:insert_block name="origin" />
+    </joint>
+    <link name="${prefix}floor">
+        <visual>
+            <geometry>
+                <box size="${length} ${width} ${height}"/>
+            </geometry>
+            <origin rpy="0 0 0" xyz="0 0 ${height/2}"/>
+            <material name="${prefix}color">
+              <xacro:insert_block name="color" />
+            </material>
+        </visual>
+    </link>
+  </xacro:macro>
 </robot>
